Commit message: updated 3D model

File: urdf_robot/urdf/rover.urdf.xacro (robot description, xacro)
@@ -38,7 +38,8 @@
   <link name="base_link">
     <visual>
-      <origin xyz="0.0 0.0 0.0" />
+      <origin xyz="0.0 0.0 -1.15" rpy="-1.57 0.0 -1.57" />
       <geometry>
-        <box size="0.5 0.43 0.02"/>
+        <mesh
+          filename="package://urdf_robot/meshes/TEST.STL" />
       </geometry>
       <material name="grey"/>
@@ -54,29 +55,8 @@
     </xacro:inertial_box>
   </link>
-  <link name="torso">
-    <visual>
-      <geometry>
-        <cylinder length="0.8" radius="0.03"/>
-      </geometry>
-      <material name="grey"/>
-    </visual>
-    <collision>
-      <geometry>
-        <cylinder length="0.8" radius="0.03"/>
-      </geometry>
-    </collision>
-    <xacro:inertial_cylinder mass="0.001" length="0.8" radius="0.03">
-      <origin xyz="0.0 0.0 0.0" rpy="0.0 0.0 0.0"/>
-    </xacro:inertial_cylinder>
-  </link>
   <joint name="base_joint" type="fixed">
     <parent link="base_footprint"/>
     <child link="base_link"/>
     <origin xyz="-0.1 0.0 0.0" rpy="0.0 0.0 0.0"/>
-  </joint>
-  <joint name="base_to_torso" type="fixed">
-    <parent link="base_link"/>
-    <child link="torso"/>
-    <origin xyz="0.0 0.0 0.4"/>
   </joint>
   <!--front right wheel-->
@@ -103,5 +83,5 @@
     <axis xyz="0 0 1"/>
     <!--limit lower="-3.14159" upper="3.14159" velocity="50.0" effort="1000.0"/-->
-    <origin xyz="0.13 0.215 0" rpy="-1.57 0 0"/>
+    <origin xyz="0.02 0.215 0" rpy="-1.57 0 0"/>
   </joint>
   <!--front left wheel-->
@@ -128,5 +108,5 @@
     <axis xyz="0 0 1"/>
     <!--limit lower="-3.14159" upper="3.14159" velocity="50.0" effort="1000.0"/-->
-    <origin xyz="0.13 -0.215 0" rpy="-1.57 0 0"/>
+    <origin xyz="0.02 -0.215 0" rpy="-1.57 0 0"/>
   </joint>
   <!--CASTER WHEEL-->
@@ -153,8 +133,5 @@
   </link>
   <gazebo reference="base_link">
-    <material>Gazebo/Blue</material>
-  </gazebo>
-  <gazebo reference="torso">
-    <material>Gazebo/Blue</material>
+    <material>Gazebo/Grey</material>
   </gazebo>
   <gazebo reference="wheel_frontr_link">
@@ -172,5 +149,5 @@
     <plugin name="differential_drive_controller" filename="libgazebo_ros_diff_drive.so">
     <!-- Plugin update rate in Hz -->
-      <updateRate>10</updateRate>
+      <!--updateRate>10</updateRate-->
     <!-- Name of left joint, defaults to `left_joint` -->
       <leftJoint>joint_frontl</leftJoint>
@@ -192,5 +169,5 @@
       <odometryFrame>odom</odometryFrame>
     <!-- Robot frame to calculate odometry from, defaults to `base_footprint` -->
-      <robotBaseFrame>base_link</robotBaseFrame>
+      <robotBaseFrame>base_footprint</robotBaseFrame>
     <!-- Odometry source, 0 for ENCODER, 1 for WORLD, defaults to WORLD -->
       <odometrySource>1</odometrySource>

Commit message: updated Lidar model

File: urdf_robot/urdf/rover.urdf.xacro (robot description, xacro)
@@ -132,4 +132,28 @@
     </xacro:inertial_sphere>
   </link>
+  <!--LIDAR-->
+  <joint name="lidar_joint" type="fixed">
+    <parent link="base_link"/>
+    <child link="lidar_link"/>
+    <origin xyz="0.0 0.0 1.14" rpy="0.0 0.0 0.0"/>
+  </joint>
+  <link name="lidar_link">
+    <visual>
+      <origin xyz="0.0 0.0 0.0" rpy="0.0 0.0 0.0"/>
+      <geometry>
+        <mesh
+          filename="package://urdf_robot/meshes/lidar_3d_v2.dae" />
+      </geometry>
+      <material name="black"/>
+    </visual>
+    <collision>
+      <geometry>
+        <cylinder radius="0.07" length="0.03"/>
+      </geometry>
+    </collision>
+    <xacro:inertial_cylinder mass="0.2" length="0.03" radius="0.07">
+      <origin xyz="0.0 0.0 0.0" rpy="0.0 0.0 0.0"/>
+    </xacro:inertial_cylinder>
+  </link>
   <gazebo reference="base_link">
     <material>Gazebo/Grey</material>
@@ -139,4 +163,7 @@
   </gazebo>
   <gazebo reference="wheel_frontl_link">
+    <material>Gazebo/Black</material>
+  </gazebo>
+  <gazebo reference="lidar_link">
     <material>Gazebo/Black</material>
   </gazebo>

Commit message: Add files via upload

File: urdf_robot/urdf/rover.urdf.xacro (robot description, xacro)
@@ -135,8 +135,8 @@
   <joint name="lidar_joint" type="fixed">
     <parent link="base_link"/>
-    <child link="lidar_link"/>
+    <child link="laser_frame"/>
     <origin xyz="0.0 0.0 1.14" rpy="0.0 0.0 0.0"/>
   </joint>
-  <link name="lidar_link">
+  <link name="laser_frame">
     <visual>
       <origin xyz="0.0 0.0 0.0" rpy="0.0 0.0 0.0"/>
@@ -165,5 +165,5 @@
     <material>Gazebo/Black</material>
   </gazebo>
-  <gazebo reference="lidar_link">
+  <gazebo reference="laser_frame">
     <material>Gazebo/Black</material>
   </gazebo>
@@ -209,3 +209,38 @@
     </plugin>
   </gazebo>
+  <gazebo reference="laser_frame">
+    <sensor type="ray" name="head_hokuyo_sensor">
+      <pose>0 0 0 0 0 0</pose>
+      <visualize>true</visualize>
+      <update_rate>10</update_rate>
+      <ray>
+        <scan>
+          <horizontal>
+            <samples>360</samples>
+            <resolution>1</resolution>
+            <min_angle>-3.14</min_angle>
+            <max_angle>3.14</max_angle>
+          </horizontal>
+        </scan>
+        <range>
+          <min>0.3</min>
+          <max>12</max>
+          <resolution>0.01</resolution>
+        </range>
+        <noise>
+          <type>gaussian</type>
+          <!-- Noise parameters based on published spec for Hokuyo laser
+               achieving "+-30mm" accuracy at range < 10m.  A mean of 0.0m and
+               stddev of 0.01m will put 99.7% of samples within 0.03m of the true
+               reading. -->
+          <mean>0.0</mean>
+          <stddev>0.01</stddev>
+        </noise>
+      </ray>
+      <plugin name="gazebo_ros_head_hokuyo_controller" filename="libgazebo_ros_laser.so">
+        <topicName>/scan</topicName>
+        <frameName>laser_frame</frameName>
+      </plugin>
+    </sensor>
+  </gazebo>
 </robot>

Commit message: added camera

File: urdf_robot/urdf/rover.urdf.xacro (robot description, xacro)
@@ -156,4 +156,25 @@
     </xacro:inertial_cylinder>
   </link>
+  <!--CAMERA-->
+  <joint name="camera_joint" type="fixed">
+    <parent link="base_link"/>
+    <child link="camera_link"/>
+    <origin xyz="0.05 0.0 1.0" rpy="0.0 0.0 0.0"/>
+  </joint>
+  <link name="camera_link">
+    <visual>
+      <origin xyz="0.0 0.0 0.0" rpy="0.0 0.0 0.0"/>
+      <geometry>
+        <box size="0.01 0.03 0.03"/>
+      </geometry>
+      <material name="black"/>
+    </visual>
+  </link>
+  <joint name="camera_optical_joint" type="fixed">
+    <parent link="camera_link"/>
+    <child link="camera_link_optical"/>
+    <origin xyz="0.0 0.0 0.0" rpy="-1.57 0.0 -1.57"/>
+  </joint>
+  <link name="camera_link_optical"></link>
   <gazebo reference="base_link">
     <material>Gazebo/Grey</material>
@@ -166,4 +187,7 @@
   </gazebo>
   <gazebo reference="laser_frame">
+    <material>Gazebo/Black</material>
+  </gazebo>
+  <gazebo reference="camera_link">
     <material>Gazebo/Black</material>
   </gazebo>
@@ -212,5 +236,5 @@
     <sensor type="ray" name="head_hokuyo_sensor">
       <pose>0 0 0 0 0 0</pose>
-      <visualize>true</visualize>
+      <visualize>false</visualize>
       <update_rate>10</update_rate>
       <ray>
@@ -244,3 +268,17 @@
     </sensor>
   </gazebo>
+  <gazebo reference="camera_link">
+    <sensor type="camera" name="camera">
+      <pose>0 0 0 0 0 0</pose>
+      <visualize>true</visualize>
+      <update_rate>10</update_rate>
+      <camera>
+      <image width="640" height="480" hfov="1.5708" format="RGB8" near="0.01" far="50.0"/>
+      </camera>
+      <plugin name="camera_controller" filename="libgazebo_ros_camera.so">
+        <!--topicName>/scan</topicName-->
+        <frameName>camera_link_optical</frameName>
+      </plugin>
+    </sensor>
+  </gazebo>
 </robot>

Commit message: Add files via upload

File: urdf_robot/urdf/rover.urdf.xacro (robot description, xacro)
@@ -51,5 +51,5 @@
       </geometry>
     </collision>
-    <xacro:inertial_box mass="20" x="0.5" y="0.43" z="0.02">
+    <xacro:inertial_box mass="5" x="0.5" y="0.43" z="0.02">
       <origin xyz="0.0 0.0 0.0" rpy="0.0 0.0 0.0"/>
     </xacro:inertial_box>
@@ -83,5 +83,5 @@
     <axis xyz="0 0 1"/>
     <!--limit lower="-3.14159" upper="3.14159" velocity="50.0" effort="1000.0"/-->
-    <origin xyz="0.02 0.215 0" rpy="-1.57 0 0"/>
+    <origin xyz="0.02 0.222 0" rpy="-1.57 0 0"/>
   </joint>
   <!--front left wheel-->
@@ -108,5 +108,5 @@
     <axis xyz="0 0 1"/>
     <!--limit lower="-3.14159" upper="3.14159" velocity="50.0" effort="1000.0"/-->
-    <origin xyz="0.02 -0.215 0" rpy="-1.57 0 0"/>
+    <origin xyz="0.02 -0.208 0" rpy="-1.57 0 0"/>
   </joint>
   <!--CASTER WHEEL-->
@@ -128,5 +128,5 @@
       </geometry>
     </collision>
-    <xacro:inertial_sphere mass="0.3" radius="0.07">
+    <xacro:inertial_sphere mass="0.1" radius="0.07">
       <origin xyz="0.0 0.0 0.0" rpy="0.0 0.0 0.0"/>
     </xacro:inertial_sphere>
@@ -214,5 +214,5 @@
       <wheelTorque>28</wheelTorque>
     <!-- Topic to receive geometry_msgs/Twist message commands, defaults to `cmd_vel` -->
-      <commandTopic>turtle1/cmd_vel</commandTopic>
+      <commandTopic>/cmd_vel</commandTopic>
     <!-- Topic to publish nav_msgs/Odometry messages, defaults to `odom` -->
       <odometryTopic>odom</odometryTopic>

Commit message: added IMU sensor

File: urdf_robot/urdf/rover.urdf.xacro (robot description, xacro)
@@ -177,4 +177,11 @@
   </joint>
   <link name="camera_link_optical"></link>
+  <!--IMU_SENSOR-->
+  <link name="imu_link"></link>
+  <joint name="imu_joint" type="fixed">
+    <parent link="base_link"/>
+    <child link="imu_link"/>
+    <origin xyz="0.0 0.0 0.0" rpy="0.0 0.0 0.0"/>
+  </joint>
   <gazebo reference="base_link">
     <material>Gazebo/Grey</material>
@@ -282,3 +289,23 @@
     </sensor>
   </gazebo>
+  <gazebo reference="imu_link">
+    <gravity>true</gravity>
+    <sensor name="imu_sensor" type="imu">
+      <always_on>true</always_on>
+      <update_rate>100</update_rate>
+      <visualize>true</visualize>
+      <topic>__default_topic__</topic>
+      <plugin filename="libgazebo_ros_imu_sensor.so" name="imu_plugin">
+        <topicName>imu</topicName>
+        <bodyName>imu_link</bodyName>
+        <updateRateHZ>10.0</updateRateHZ>
+        <gaussianNoise>0.0</gaussianNoise>
+        <xyzOffset>0 0 0</xyzOffset>
+        <rpyOffset>0 0 0</rpyOffset>
+        <frameName>imu_link</frameName>
+        <initialOrientationAsReference>false</initialOrientationAsReference>
+      </plugin>
+      <pose>0 0 0 0 0 0</pose>
+    </sensor>
+  </gazebo>
 </robot>

Commit message: Add files via upload

File: urdf_robot/urdf/rover.urdf.xacro (robot description, xacro)
@@ -83,5 +83,5 @@
     <axis xyz="0 0 1"/>
     <!--limit lower="-3.14159" upper="3.14159" velocity="50.0" effort="1000.0"/-->
-    <origin xyz="0.02 0.222 0" rpy="-1.57 0 0"/>
+    <origin xyz="0.02 0.222 0" rpy="1.57 0 0"/>
   </joint>
   <!--front left wheel-->
@@ -108,5 +108,5 @@
     <axis xyz="0 0 1"/>
     <!--limit lower="-3.14159" upper="3.14159" velocity="50.0" effort="1000.0"/-->
-    <origin xyz="0.02 -0.208 0" rpy="-1.57 0 0"/>
+    <origin xyz="0.02 -0.208 0" rpy="1.57 0 0"/>
   </joint>
   <!--CASTER WHEEL-->
@@ -221,5 +221,5 @@
       <wheelTorque>28</wheelTorque>
     <!-- Topic to receive geometry_msgs/Twist message commands, defaults to `cmd_vel` -->
-      <commandTopic>/cmd_vel</commandTopic>
+      <commandTopic>turtle1/cmd_vel</commandTopic>
     <!-- Topic to publish nav_msgs/Odometry messages, defaults to `odom` -->
       <odometryTopic>odom</odometryTopic>
@@ -297,5 +297,5 @@
       <topic>__default_topic__</topic>
       <plugin filename="libgazebo_ros_imu_sensor.so" name="imu_plugin">
-        <topicName>imu</topicName>
+        <topicName>imu_data</topicName>
         <bodyName>imu_link</bodyName>
         <updateRateHZ>10.0</updateRateHZ>
